File: hardware/backbone/backbone.kicad_sch (KiCad schematic)
At the start: 84 parts, among them J1 RESET, J10 CORE_A, J11 MOUNT, J12 PW, J13 FIELD_B, J14 FIELD_A, J15 UART PROG, J16 ALED, J2 FROM_PREVIOUS, J4 FROM_PREVIOUS, J5 CONN_A, J6 BOOTLOADER, J7 CONN_B, J8 CORE_B, J9 TO NEXT, Q2 AO3401A, U11 470nH DCR=450m, U13 470nH DCR=450m, U15 ST25R100, U17 BLM18PG471SZ1D, U2 SN65HVD230DR, U4 AP2112K-3.3TRG1, U5 ESP32-C3-MINI-1-H4X, U8 G3VM-61VY3, U9 SN74AHCT1G14DCKR, X1 NX2016SA 27.12MHz

Commit message: added usb c to backbone, changed esp32 c3 to esp32 s3 so no more core needed to power the board and program it
Parts:
- removed C12, C22: 100nF, SpaghettiLAB2:C0603, symbol STMICRO:root_1_GRM033C71A104KE14D_STMICRO.SchLib
- removed C3, C7: 100nF, SpaghettiLAB2:C0603, symbol Device:C
- removed J1: RESET, Connector_PinHeader_2.54mm:PinHeader_1x02_P2.54mm_Vertical, symbol Connector:Conn_01x02_Pin
- removed J12: PW, Connector_PinHeader_2.54mm:PinHeader_1x02_P2.54mm_Vertical, symbol Connector:Conn_01x02_Pin
- removed J15: UART PROG, Connector_PinHeader_2.54mm:PinHeader_1x02_P2.54mm_Vertical, symbol Connector:Conn_01x02_Pin
- removed J16: ALED, Connector_PinSocket_2.54mm:PinSocket_1x03_P2.54mm_Vertical, symbol Connector:Conn_01x03_Pin
- removed J6: BOOTLOADER, Connector_PinHeader_2.54mm:PinHeader_1x02_P2.54mm_Vertical, symbol Connector:Conn_01x02_Pin
- removed JP1: FIRST_PROG, Jumper:SolderJumper-2_P1.3mm_Open_RoundedPad1.0x1.5mm, symbol Jumper:Jumper_2_Open
- removed LED1: SK6812MINI-E, SpaghettiLAB2:LED-SMD_4P-L3.2-W2.8-LS5.9_SK6812MINI-E, symbol USBC_PD_mo-easyedapro:SK6812MINI-E_C5149201
- removed R1, R2: 4.7k, SpaghettiLAB2:R0603, symbol Device:R
- removed R9: 220R, SpaghettiLAB2:R0603, symbol Device:R
- removed U5: ESP32-C3-MINI-1-H4X, SpaghettiLAB:WIFIM-SMD_ESP32-C3-MINI-1, symbol SpaghettiLAB:ESP32-C3-MINI-1-H4X
- removed U9: SN74AHCT1G14DCKR, SpaghettiLAB2:SOT-353_L2.2-W1.4-P0.65-LS2.4-BR, symbol USBC_PD_mo-easyedapro:SN74AHCT1G14DCKR
- added C73, C74: 100nF, SpaghettiLAB:C0603, symbol Device:C
- added D2, D3, D5: LED, SpaghettiLAB:LED0603-RD, symbol Device:LED
- added D4: SS54_C22452, SpaghettiLAB:SMA_L4.4-W2.8-LS5.4-R-RD, symbol SpaghettiLAB:SS54_C22452
- added R15, R16: 4.7k, SpaghettiLAB:R0603, symbol Device:R
- added R17, R18: 33R, SpaghettiLAB:R0603, symbol Device:R
- added R20, R23: 5.1k, SpaghettiLAB:R0603, symbol Device:R
- added R21, R22, R24: 330R, SpaghettiLAB:R0603, symbol Device:R
- added TP12, TP13, TP15, TP18, TP19, TP21, TP8, TP9: SMD/0.6mm, TestPoint:TestPoint_Pad_D1.0mm, symbol STMICRO:root_3_PLAGE-CMS-DIAM-0.6mm_STMICRO.SchLib
- added U19: ESP32-S3-MINI-1, RF_Module:ESP32-S2-MINI-1, symbol RF_Module:ESP32-S3-MINI-1
- added USB1: TYPEC-324G-BCP24, SpaghettiLAB:USB-C-SMD_TYPEC-324G-BCP24, symbol SpaghettiLAB:TYPEC-324G-BCP24
Connections:
- net 5V: now also D4.2 (K), R22.1
- net CAN_RX: now also U19.8 (IO4)
- net CAN_TX: now also U19.9 (IO5)
- net GND: now also C73.2, C74.1, D2.1 (K), D3.1 (K), R20.2, R23.1, TP12.1, TP13.1, TP21.1, U19.1 (GND), U19.2 (GND), U19.42 (GND), U19.43 (GND), U19.46 (GND), U19.47 (GND), U19.48 (GND), U19.49 (GND), U19.50 (GND), U19.51 (GND), U19.52 (GND), U19.53 (GND), U19.54 (GND), U19.55 (GND), U19.56 (GND), U19.57 (GND), U19.58 (GND), U19.59 (GND), U19.60 (GND), U19.61 (GND), U19.62 (GND), U19.63 (GND), U19.64 (GND), U19.65 (GND), USB1.1 (EP), USB1.2 (EP), USB1.3 (EP), USB1.4 (EP), USB1.A1 (GND), USB1.A12 (GND), USB1.B1 (GND), USB1.B12 (GND)
- net VCORE: now also C74.2, R15.1, R16.1, R21.1, R24.1, TP15.1, U19.3 (3V3)
- net RFI1_25R200 renamed RFI1_25R100
- net RFI2_25R200 renamed RFI2_25R100
- net RFO1_25R200 renamed RFO1_25R100
- net RFO2_25R200 renamed RFO2_25R100
- new net: D5.2 (A), R24.2
- new net: D2.2 (A), R21.2
- new net: R23.2, USB1.A5 (CC1)
- new net: R20.1, USB1.B5 (CC2)
- new net: R18.2, U19.23 (USB_D-)
- new net: R17.2, U19.24 (USB_D+)
- new net: D3.2 (A), R22.2
- new net BOOT: R15.2, TP9.1, U19.4 (IO0)
- new net IO1: U19.5 (IO1)
- new net IO10: U19.14 (IO10)
- new net IO11: U19.15 (IO11)
- new net IO12: U19.16 (IO12)
- new net IO13: U19.17 (IO13)
- new net IO14: U19.18 (IO14)
- new net IO15: U19.19 (IO15)
- new net IO16: U19.20 (IO16)
- new net IO17: U19.21 (IO17)
- new net IO18: U19.22 (IO18)
- new net IO2: U19.6 (IO2)
- new net IO21: U19.25 (IO21)
- new net IO26: U19.26 (IO26)
- new net IO3: U19.7 (IO3)
- new net IO33: U19.28 (IO33)
- new net IO35: U19.31 (IO35)
- new net IO36: U19.32 (IO36)
- new net IO37: U19.33 (IO37)
- new net IO38: U19.34 (IO38)
- new net IO39: U19.35 (IO39)
- new net IO40: U19.36 (IO40)
- new net IO41: U19.37 (IO41)
- new net IO42: U19.38 (IO42)
- new net IO45: U19.41 (IO45)
- new net IO46: U19.44 (IO46)
- new net IO47: U19.27 (IO47)
- new net IO48: U19.30 (IO48)
- new net RXD0: TP18.1, U19.40 (RXD0)
- new net STATUS: D5.1 (K), U19.29 (IO34)
- new net TXD0: TP19.1, U19.39 (TXD0)
- new net USB_D+: R17.1, USB1.A6 (DP1), USB1.B6 (DP2)
- new net USB_D-: R18.1, USB1.A7 (DN1), USB1.B7 (DN2)
- new net VBUS: D4.1 (A), USB1.A4 (VBUS), USB1.A9 (VBUS), USB1.B4 (VBUS), USB1.B9 (VBUS)
- new net ~{RESET}: C73.1, R16.2, TP8.1, U19.45 (EN)
- no-connect marks 27 -> 22
Other:
- note added: "LEDs"
- note added: "USB"
- note removed: "FIRST PROG: UART OVER CAN BRIDGE OPEN"
- note removed: "NB: INVERTING OUTPUT!!!"
- note removed: "SLOT STATUS ADDRESSABLE LED"
- moved on the sheet: ANT1, ANT2, C1, C13, C16, C18, C20, C23, C28, C30, C32, C33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

Commit message: board with usb and esp32 s3 completely routed
Parts:
- removed TP10, TP14, TP6: SMD/0.6mm, TestPoint:TestPoint_Pad_D1.0mm, symbol STMICRO:root_1_PLAGE-CMS-DIAM-0.6mm_STMICRO.SchLib
- removed TP11, TP16, TP7: SMD/0.6mm, TestPoint:TestPoint_Pad_D1.0mm, symbol STMICRO:root_3_PLAGE-CMS-DIAM-0.6mm_STMICRO.SchLib
Connections:
- net IO1 is gone; now on net NFC_RST: U19.5 (IO1)
- net IO10 is gone; now on net STATUS: U19.14 (IO10)
- net IO2 is gone; now on net NFC_CS: U19.6 (IO2)
- net IO3 is gone; now on net NFC_MOSI: U19.7 (IO3)
- net IO35 is gone; now on net A3: U19.31 (IO35)
- net IO36 is gone; now on net A2: U19.32 (IO36)
- net IO37 is gone; now on net A1: U19.33 (IO37)
- net IO38 is gone; now on net A0: U19.34 (IO38)
- net IO48 is gone; now on net CAN_TX: U19.30 (IO48)
- net 5V: now also Q2.2 (S); no longer Q2.3 (D)
- net CAN_RX: now also U19.29 (IO34); no longer U19.8 (IO4)
- net CAN_TX: no longer U19.9 (IO5)
- net NFC_IRQ: now also U19.9 (IO5)
- net NFC_MISO: now also U19.10 (IO6)
- net NFC_SCK: now also U19.8 (IO4)
- net STATUS: no longer U19.29 (IO34)
- net at R5.2: now also Q2.3 (D); no longer Q2.2 (S)
- net IO7: now reaches U19.11 (IO7)
- net IO8: now reaches U19.12 (IO8)
- net IO9: now reaches U19.13 (IO9)
Other:
- moved on the sheet: R20, R23

Commit message: fix backbone schematic connectivity and power flags
Parts:
- C1, C13, C16, C18, C20, C23, C28, C30, C32, C33, C35, C37, C39, C41, C43, C46, C48, C5, C51, C54, C55, C58, C60, C62, C63, C65, C70, C72, C9: footprint SpaghettiLAB2:C0603 -> SpaghettiLAB:C0603
- R11, R14, R4, R5, R8: footprint SpaghettiLAB2:R0603 -> SpaghettiLAB:R0603
- U4: footprint SpaghettiLAB2:SOT-25-5_L2.9-W1.6-P0.95-LS2.8-BL -> SpaghettiLAB:SOT-25-5_L2.9-W1.6-P0.95-LS2.8-BL
Connections:
- net Net-(D5-A): now reaches D5.2 (A), R24.2
- net Net-(ANT1-Pad2): now reaches ANT1.2, R14.2
- net Net-(U15-VDD): now reaches C58.2, C62.2, U15.7 (VDD), U17.1
- net Net-(C32-Pad2): now reaches C32.2, C54.1, C55.2, R14.1
- net Net-(R5-Pad1): now reaches R5.1, U8.1
- net Net-(Q2-D): now reaches Q2.3 (D), R5.2
- net Net-(D2-A): now reaches D2.2 (A), R21.2
- net Net-(USB1-CC1): now reaches R23.2, USB1.A5 (CC1)
- net Net-(USB1-CC2): now reaches R20.1, USB1.B5 (CC2)
- net Net-(ANT2-Pad2): now reaches ANT2.2, R11.2
- net Net-(C28-Pad2): now reaches C28.2, C43.1, C46.2, R11.1
- net Net-(U19-USB_D-): now reaches R18.2, U19.23 (USB_D-)
- net Net-(U19-USB_D+): now reaches R17.2, U19.24 (USB_D+)
- net Net-(R8-Pad2): now reaches R8.2, U8.3
- net Net-(D3-A): now reaches D3.2 (A), R22.2

Commit message: software fixes and harwdrae text to remind to route ADC pins next rev
Other:
- note added: "ADC GPIO1 - GPIO10 NEXT REVIEW NEEDS THIS MODS"

Commit message: Added text reminder for adc pins
Other:
- note added: "| ADC | Channels | GPIO | | ADC1 | CH0-CH9 | **GPIO1-GPIO10** | | ADC2 | CH0-CH9 | **GPIO11-GPIO20** | NEXT REVIEW NEEDS THIS MODS"
- note removed: "ADC GPIO1 - GPIO10 NEXT REVIEW NEEDS THIS MODS"
Changed lines of the file:
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@@
 		)
 	)
-	(text "ADC GPIO1 - GPIO10 \nNEXT REVIEW NEEDS THIS MODS"
+	(text "| ADC | Channels | GPIO |\n| ADC1 | CH0-CH9 | **GPIO1-GPIO10** |\n| ADC2 | CH0-CH9 | **GPIO11-GPIO20** |\nNEXT REVIEW NEEDS THIS MODS"
 		(exclude_from_sim no)
 		(at 77.47 205.74 0)
