File: hardware/backbone/backbone.kicad_sch (KiCad schematic)
At the start: 93 parts, among them J1 M20-7810645R, J140 M20-7810645R, J2 FROM_PREVIOUS, J3 M20-7810645R, J4 SM04B-SRSS-TB(LF)(SN), J5 FH12-24S-0.5SH(55), J9 TO NEXT, Q2 AO3401A, Q3 AO6604, Q4 AO6604, Q5 AO6604, Q6 AO6604, Q7 AO6604, Q8 AO6604, U1 ESP32-S3-WROOM-1_1U_FlexyPin_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, U10 ME6211C15M5G-N, U11 XL9535QF24, U2 SN65HVD230DR, U3 HC-TYPE-C-16P-01A, U4 TPS562201DDCR, U8 G3VM-61VY3, U9 ME6211C28M5G-N

Commit message: Add AG32 universal supervisor schematic and LCSC CAD assets
Parts:
- removed C87: 100nF, SpaghettiLAB:C0603, symbol Device:C
- removed U11: XL9535QF24, LCSC_Ports:QFN-24_L4.0-W4.0-P0.50-BL-EP2.6, symbol SpaghettiLAB:XL9535QF24_6Ports
- added C88, C89: 100nF, SpaghettiLAB:C0603, symbol Device:C
- added R50, R51, R52, R53, R54, R55: 100k, SpaghettiLAB:R0603, symbol Device:R
- added R56, R57, R58, R59, R60, R61: 0.1R, Resistor_SMD:R_1206_3216Metric, symbol Device:R
- added U12, U13: SN74CBTLV3125PWR, LCSC_Ports:TSSOP-14_L5.0-W4.4-P0.65-LS6.4-BL, symbol SpaghettiLAB:SN74CBTLV3125_4Switches
- Q3, Q4, Q5, Q6, Q7, Q8, R38, R39, R40, R41, R42, R43, R44, R45, R46, R47, R48, R49: Assembly (none) -> AG32
- R17, R18: value 33R -> 33R DNP / ESP USB; Assembly (none) -> ESP_USB_ONLY; now not fitted
Connections:
- net 5V: no longer J3.2
- net A0: now also J3.3, U12.2 (A); no longer J1.1, J1.2, J140.1, J140.2, J3.6, Q3.4 (D), Q3.6 (D)
- net A1: now also J3.4, U12.5 (A); no longer J1.3, J1.4, J140.3, J140.4, J3.8, Q4.4 (D), Q4.6 (D)
- net A2: now also J3.7, U12.9 (A); no longer J1.5, J1.6, J140.5, J140.6, J3.10, Q5.4 (D), Q5.6 (D)
- net A3: now also J3.8, U12.12 (A); no longer J1.7, J1.8, J140.7, J140.8, J3.12, Q6.4 (D), Q6.6 (D)
- net A4: now also U1.39 (IO1), U13.2 (A); no longer J1.10, J1.9, J140.10, J140.9, Q7.4 (D), Q7.6 (D), U1.19 (IO11)
- net A5: now also J3.12, U1.38 (IO2), U13.5 (A); no longer J1.11, J1.12, J140.11, J140.12, J3.9, Q8.4 (D), Q8.6 (D), U1.20 (IO12)
- net ALED: no longer U1.9 (IO16)
- net CAN_RX: no longer U1.24 (IO47)
- net CAN_TX: no longer U1.25 (IO48)
- net GND: now also J3.10, J3.2, J3.6, C88.2, C89.2, U12.7 (GND), U13.7 (GND); no longer J3.3, J3.4
- net VCORE: now also J3.5, J3.9, C88.1, C89.1, R50.1, R51.1, R52.1, R53.1, R54.1, R55.1, U12.14 (VCC), U13.13 (~{OE}), U13.14 (VCC)
- net P_GATE_1: now reaches Q4.3 (G), R40.2
- net N_GATE_1: now reaches Q4.1 (G), R41.1
- net N_GATE_2: now reaches Q5.1 (G), R43.1
- net N_GATE_5: now reaches Q8.1 (G), R49.1
- net P_GATE_5: now reaches Q8.3 (G), R48.2
- net N_GATE_0: now reaches Q3.1 (G), R39.1
- net P_GATE_4: now reaches Q7.3 (G), R46.2
- net N_GATE_3: now reaches Q6.1 (G), R45.1
- net P_GATE_3: now reaches Q6.3 (G), R44.2
- net P_GATE_2: now reaches Q5.3 (G), R42.2
- net P_GATE_0: now reaches Q3.3 (G), R38.2
- net N_GATE_4: now reaches Q7.1 (G), R47.1
- net A6 renamed CTRL13
- net CTRL13: no longer J3.7
- net A7 renamed CTRL14
- net CTRL14: no longer J3.5
- net IO1 renamed IO11
- net IO11: now also U1.19 (IO11); no longer U1.39 (IO1)
- net IO15: no longer names the net of U1.8 (IO15)
- net IO15: no longer R30.1
- net IO2 renamed IO12
- net IO12: now also U1.20 (IO12); no longer U1.38 (IO2)
- net RXD0 renamed SPI_MISO
- net TXD0 renamed SPI_MOSI
- new net DAC_BYPASS_N: U13.10 (~{OE})
- new net DAC_LIMITED: U13.8 (B)
- new net DAC_RAW: U13.9 (A)
- new net ISO_A0_N: R50.2, U12.1 (~{OE})
- new net ISO_A1_N: R51.2, U12.4 (~{OE})
- new net ISO_A2_N: R52.2, U12.10 (~{OE})
- new net ISO_A3_N: R53.2, U12.13 (~{OE})
- new net ISO_A4_N: R54.2, U13.1 (~{OE})
- new net ISO_A5_N: R55.2, U13.4 (~{OE})
- new net N_A0: Q3.4 (D), Q3.6 (D), R56.1, U12.3 (B)
- new net N_A1: Q4.4 (D), Q4.6 (D), R57.1, U12.6 (B)
- new net N_A2: Q5.4 (D), Q5.6 (D), R58.1, U12.8 (B)
- new net N_A3: Q6.4 (D), Q6.6 (D), R59.1, U12.11 (B)
- new net N_A4: Q7.4 (D), Q7.6 (D), R60.1, U13.3 (B)
- new net N_A5: Q8.4 (D), Q8.6 (D), R61.1, U13.6 (B)
- new net PORT_A0: J1.1, J1.2, J140.1, J140.2, R56.2
- new net PORT_A1: J1.3, J1.4, J140.3, J140.4, R57.2
- new net PORT_A2: J1.5, J1.6, J140.5, J140.6, R58.2
- new net PORT_A3: J1.7, J1.8, J140.7, J140.8, R59.2
- new net PORT_A4: J1.10, J1.9, J140.10, J140.9, R60.2
- new net PORT_A5: J1.11, J1.12, J140.11, J140.12, R61.2
- new net TERM_CTRL: R30.1
- no-connect marks 11 -> 12
Other:
- added sheet AG32 supervisor e strumenti (ports-ag32.kicad_sch)
- note added: "A0-A5 = lato micro/J3; PORT_A0-A5 = lato MOSFET e J1/J140. Default aperto."
- note added: "AG32 firmware: set all GPIO Hi-Z, disable both MOSFETs before switching modes. Analog bypass remains U12/U13."
- note added: "AG32 universal board: ESP32 optional. See AG32 supervisor sheet and AG32-SUPERVISOR.md. Old TI/Q32 variants superseded on this branch."
- note added: "GPIO mode: /OE=0, P=OFF, N=OFF. 3V3/GND mode: /OE=1 prima di abilitare il MOSFET."
- note added: "ISOLAMENTO BIDIREZIONALE J3 <-> J1/J140 — /OE=1 APERTO, /OE=0 COLLEGATO"
- note added: "J1/J140: PORT_A0-A5. J3: lato micro diretto. GPIO13/14: comandi isolamento."
- note added: "J3: 3V3/GND + A0/A1; 3V3/GND + A2/A3; 3V3/GND + A4/A5"
- note added: "PORT_A4 / GPIO1 — FILA 5"
- note added: "PORT_A5 / GPIO2 — FILA 6"
- note removed: "A4 / GPIO11 — FILA 5"
- note removed: "A5 / GPIO12 — FILA 6"
- note removed: "Firmware: prima GPIO in ingresso; spegnere entrambi i MOSFET prima di cambiare modo."
- note removed: "J1 e J140: coppie di contatti della stessa fila in comune. A6/A7 invariati."

Commit message: Use AG32 internal converters and place backbone hardware
Parts:
- removed C75, C76, C77, C78: 4.7uF/10V X7R, SpaghettiLAB:C0603, symbol Device:C
- removed C79, C80, C81, C83: 100nF, SpaghettiLAB:C0603, symbol Device:C
- removed J5: FH12-24S-0.5SH(55), SpaghettiLAB:Hirose_FH12-24S-0.5SH_1x24-1MP_P0.50mm_Horizontal, symbol SpaghettiLAB:FPC_24_Hirose_FH12
- removed R28, R29: 10k, SpaghettiLAB:R0603, symbol Device:R
- removed R30: 0, SpaghettiLAB:R0603, symbol Device:R
- removed R31, R32, R33, R34, R35: 0R, Resistor_SMD:R_0603_1608Metric_Pad0.98x0.95mm_HandSolder, symbol Device:R
- removed U10: ME6211C15M5G-N, Package_TO_SOT_SMD:SOT-23-5, symbol SpaghettiLAB:ME6211C15M5G-N
- removed U9: ME6211C28M5G-N, Package_TO_SOT_SMD:SOT-23-5, symbol SpaghettiLAB:ME6211C28M5G-N
- added C100, C101, C119, C121, C122, C123, C124, C90, C91, C92, C93, C94, C95, C96, C97, C98: 100nF, Capacitor_SMD:C_0603_1608Metric, symbol Device:C
- added C99: 1uF, Capacitor_SMD:C_0603_1608Metric, symbol Device:C
- added R100, R101, R102, R98, R99: 0R / ESP-only, Resistor_SMD:R_0603_1608Metric, symbol Device:R
- added R70, R71, R74, R75, R76, R78: 100k, Resistor_SMD:R_0603_1608Metric, symbol Device:R
- added R72, R73, R83, R84: 10k, Resistor_SMD:R_0603_1608Metric, symbol Device:R
- added R77: 4.7k 0.1% 25ppm, Resistor_SMD:R_0603_1608Metric, symbol Device:R
- added R79, R80: 4.7k, Resistor_SMD:R_0603_1608Metric, symbol Device:R
- added R81, R82: 22R DNP / AG USB, Resistor_SMD:R_0603_1608Metric, symbol Device:R
- added R85, R86, R87, R88: 1k, Resistor_SMD:R_0603_1608Metric, symbol Device:R
- added TP22: AG_NRST, TestPoint:TestPoint_Pad_D1.0mm, symbol Connector:TestPoint
- added TP23: AG_JTMS, TestPoint:TestPoint_Pad_D1.0mm, symbol Connector:TestPoint
- added TP24: AG_JTCK, TestPoint:TestPoint_Pad_D1.0mm, symbol Connector:TestPoint
- added TP25: AG_JTDI, TestPoint:TestPoint_Pad_D1.0mm, symbol Connector:TestPoint
- added TP26: AG_JTDO, TestPoint:TestPoint_Pad_D1.0mm, symbol Connector:TestPoint
- added TP27: AG_JNTRST, TestPoint:TestPoint_Pad_D1.0mm, symbol Connector:TestPoint
- added TP41: DAC1_SPARE, TestPoint:TestPoint_Pad_D1.0mm, symbol Connector:TestPoint
- added TP42: SPARE_IO_17, TestPoint:TestPoint_Pad_D1.0mm, symbol Connector:TestPoint
- added TP43: SPARE_IO_33, TestPoint:TestPoint_Pad_D1.0mm, symbol Connector:TestPoint
- added TP44: SPARE_IO_34, TestPoint:TestPoint_Pad_D1.0mm, symbol Connector:TestPoint
- added TP45: ISO4_CTRL, TestPoint:TestPoint_Pad_D1.0mm, symbol Connector:TestPoint
- added TP46: ISO5_CTRL, TestPoint:TestPoint_Pad_D1.0mm, symbol Connector:TestPoint
- added TP47: AG_UART_RX, TestPoint:TestPoint_Pad_D1.0mm, symbol Connector:TestPoint
- added TP48: AG_UART_TX, TestPoint:TestPoint_Pad_D1.0mm, symbol Connector:TestPoint
- added TP49: AG_BOOT0, TestPoint:TestPoint_Pad_D1.0mm, symbol Connector:TestPoint
- added U14: AG32VF407VGT6, LCSC_Ports:LQFP-100_L14.0-W14.0-P0.50-LS16.0-TL, symbol LCSC_Ports:AG32VF407VGT6_Functional
- added U16: INA226AIDGSR, LCSC_Ports:MSOP-10_L3.0-W3.0-P0.50-LS5.0-BL, symbol LCSC_Ports:INA226AIDGSR
- added U17, U18, U19: 74HC4051BQ,115, LCSC_Ports:DHVQFN-16_L3.5-W2.5-P0.50-BL-EP, symbol LCSC_Ports:74HC4051BQ,115
- added U25: TCA9535PWR(UMW), LCSC_Ports:TSSOP-24_L7.8-W4.4-P0.65-LS6.4-BL, symbol LCSC_Ports:TCA9535PWR
- added X1: 20MHz, LCSC_Ports:OSC-SMD_4P-L3.2-W2.5-BL, symbol LCSC_Ports:SG-8018CE-20.000000MHZ-TJHPA
- R15, R16: LCSC (none) -> C25804
- R17, R18: value 33R DNP / ESP USB -> 33R / ESP USB; Assembly ESP_USB_ONLY -> FIT; now fitted
- R56, R57, R58, R59, R60, R61: Assembly Measured / 0R Basic -> LAB:0.1R / BASE:0R
Connections:
- net A0: now also U14.38 (ESP_A0)
- net A1: now also U14.39 (ESP_A1)
- net A2: now also U14.40 (ESP_A2)
- net A3: now also U14.41 (ESP_A3)
- net A4: now also U14.42 (ESP_A4)
- net A5: now also U14.43 (ESP_A5)
- net ALED: now also R102.2, U14.7 (LED_DATA)
- net CAN_RX: now also R101.2, U14.93 (CAN_RX)
- net CAN_TX: now also R100.2, U14.92 (CAN_TX)
- net CTRL13: now also R74.2, R98.1, U14.86 (SPI_CS_N)
- net CTRL14: now also R99.1, U14.87 (SPI_SCLK)
- net DAC_BYPASS_N: now also R78.2, U14.85 (DAC_BYPASS_N)
- net DAC_LIMITED: now also R77.2, U14.16 (SCAN_ADC_LIMITED), U19.3 (Z)
- net DAC_RAW: now also R77.1, U14.15 (SCAN_ADC_RAW), U14.29 (DAC0_SCAN)
- net GND: now also C100.2, C101.2, C119.2, C121.2, C122.2, C123.2, C124.2, C90.2, C91.2, C92.2, C93.2, C94.2, C95.2, C96.2, C97.2, C98.2, C99.2, R83.1, R84.1, U14.10 (VSS33), U14.20 (VSSA), U14.27 (VSS33), U14.74 (VSS33), U14.99 (VSS33), U16.1 (A1), U16.2 (A0), U16.7 (GND), U17.7 (VEE), U17.8 (GND), U18.7 (VEE), U18.8 (GND), U19.7 (VEE), U19.8 (GND), U25.12 (GND), U25.2 (A1), U25.21 (A0), U25.3 (A2), X1.2 (GND)
- net IO3: now also R75.2, U14.97 (ESP_IRQ_N)
- net IO4: now also U14.95 (EXT_I2C_SDA), U25.23 (SDA)
- net IO5: now also U14.96 (EXT_I2C_SCL), U25.22 (SCL)
- net ISO_A0_N: now also U14.64 (ISO0_N), U25.17 (P14)
- net ISO_A1_N: now also U14.65 (ISO1_N), U25.18 (P15)
- net ISO_A2_N: now also U14.66 (ISO2_N), U25.19 (P16)
- net ISO_A3_N: now also U14.67 (ISO3_N), U25.20 (P17)
- net ISO_A4_N: now also R98.2, TP45.1, U14.35 (ISO4_N)
- net ISO_A5_N: now also R99.2, TP46.1, U14.36 (ISO5_N)
- net N_A0: now also U14.44 (DRIVE_A0), U17.13 (Y0), U19.13 (Y0)
- net N_A1: now also U14.45 (DRIVE_A1), U17.14 (Y1), U19.14 (Y1)
- net N_A2: now also U14.46 (DRIVE_A2), U17.15 (Y2), U19.15 (Y2)
- net N_A3: now also U14.47 (DRIVE_A3), U17.12 (Y3), U19.12 (Y3)
- net N_A4: now also U14.48 (DRIVE_A4), U17.1 (Y4), U19.1 (Y4)
- net N_A5: now also U14.51 (DRIVE_A5), U17.5 (Y5), U19.5 (Y5)
- net N_GATE_0: now also U14.53 (N_GATE0), U25.5 (P01)
- net N_GATE_1: now also U14.55 (N_GATE1), U25.7 (P03)
- net N_GATE_2: now also U14.57 (N_GATE2), U25.9 (P05)
- net N_GATE_3: now also U14.59 (N_GATE3), U25.11 (P07)
- net N_GATE_4: now also U14.61 (N_GATE4), U25.14 (P11)
- net N_GATE_5: now also U14.63 (N_GATE5), U25.16 (P13)
- net PORT_A0: now also U14.23 (ADC_A0/IN0), U18.13 (Y0)
- net PORT_A1: now also U14.24 (ADC_A1/IN1), U18.14 (Y1)
- net PORT_A2: now also U14.25 (ADC_A2/IN2), U18.15 (Y2)
- net PORT_A3: now also U14.26 (ADC_A3/IN3), U18.12 (Y3)
- net PORT_A4: now also U14.31 (ADC_A4/IN6), U18.1 (Y4)
- net PORT_A5: now also U14.32 (ADC_A5/IN7), U18.5 (Y5)
- net P_GATE_0: now also U14.52 (P_GATE0_N), U25.4 (P00)
- net P_GATE_1: now also U14.54 (P_GATE1_N), U25.6 (P02)
- net P_GATE_2: now also U14.56 (P_GATE2_N), U25.8 (P04)
- net P_GATE_3: now also U14.58 (P_GATE3_N), U25.10 (P06)
- net P_GATE_4: now also U14.60 (P_GATE4_N), U25.13 (P10)
- net P_GATE_5: now also U14.62 (P_GATE5_N), U25.15 (P12)
- net SPI_MISO: now also R101.1, U14.91 (SPI_MISO)
- net SPI_MOSI: now also R100.1, U14.88 (SPI_MOSI)
- net TERM_CTRL: now also U14.1 (SPARE_CTRL)
- net USB_D+: now also R82.2
- net USB_D-: now also R81.2
- net VCORE: now also C100.1, C101.1, C119.1, C121.1, C122.1, C123.1, C124.1, C90.1, C91.1, C93.1, C94.1, C95.1, C96.1, C97.1, C98.1, C99.1, R70.1, R71.1, R72.1, R73.1, R74.1, R75.1, R76.1, R78.1, R79.1, R80.1, U14.100 (VDD33), U14.11 (VDD33), U14.21 (VREFP), U14.22 (VDDA), U14.28 (VDD33), U14.50 (VDD33), U14.6 (VBAT), U14.75 (VDD33), U16.6 (VS+), U17.16 (VCC), U17.17 (EP_VCC), U18.16 (VCC), U18.17 (EP_VCC), U19.16 (VCC), U19.17 (EP_VCC), U25.24 (VCC), X1.1 (OE/#ST), X1.4 (VCC)
- net ~{RESET}: now also U14.98 (ESP_RESET_OD)
- net LED_CHAIN_1: now reaches LED1.4 (DOUT), LED2.2 (DIN)
- net LED_CHAIN_2: now reaches LED2.4 (DOUT), LED3.2 (DIN)
- net LED_CHAIN_3: now reaches LED3.4 (DOUT), LED4.2 (DIN)
- net LED_CHAIN_4: now reaches LED4.4 (DOUT), LED5.2 (DIN)
- net BUCK_SW: now reaches C84.2, L1.1, U4.2 (SW)
- net USB_CC1: now reaches U3.A5 (CC1)
- net USB_CC1: now also R22.1; no longer R27.2
- net USB_CC2: now reaches U3.B5 (CC2)
- net USB_CC2: now also R27.2; no longer R22.1
- net LED_CHAIN_5: now reaches LED5.4 (DOUT), LED6.2 (DIN)
- net BUCK_FB: now reaches R36.2, R37.1, U4.4 (VFB)
- net BUCK_BOOT: now reaches C84.1, U4.6 (VBST)
- net ESP_PROG_TX: now reaches U1.24 (IO47)
- net ESP_PROG_TX: now also R102.1, R85.1
- net ESP_PROG_RX: now reaches U1.25 (IO48)
- net ESP_PROG_RX: now also R86.2
- net ESP_AG_BOOT0: now reaches U1.8 (IO15)
- net ESP_AG_BOOT0: now also R87.1
- net ESP_AG_RESET_N: now reaches U1.9 (IO16)
- net ESP_AG_RESET_N: now also R88.1
- new net AG_BOOT0: R83.2, R87.2, TP49.1, U14.94 (BOOT0)
- new net AG_BOOT1: R84.2, U14.37 (BOOT1)
- new net AG_BOOT_UART_RX: R85.2, TP47.1, U14.69 (BOOT_UART0_RX)
- new net AG_BOOT_UART_TX: R86.1, TP48.1, U14.68 (BOOT_UART0_TX)
- new net AG_JNTRST_N: R73.2, TP27.1, U14.90 (JNTRST_N)
- new net AG_JTCK: TP24.1, U14.76 (JTCK)
- new net AG_JTDI: TP25.1, U14.77 (JTDI)
- new net AG_JTDO: TP26.1, U14.89 (JTDO)
- new net AG_JTMS: TP23.1, U14.72 (JTMS)
- new net AG_NRST_N: C92.1, R72.2, R88.2, TP22.1, U14.14 (NRST_N)
- new net AG_USB_DM: R81.1, U14.70 (USB_DM)
- new net AG_USB_DP: R82.1, U14.71 (USB_DP)
- new net CLK20M: U14.12 (OSC_IN), U14.18 (CLK20M_FPGA), X1.3 (OUT)
- new net DAC1_SPARE: TP41.1, U14.30 (DAC1_SPARE)
- new net DAC_INHIBIT: R71.2, U14.81 (DAC_INHIBIT), U19.6 (E_INHIBIT)
- new net DAC_S0: U14.78 (DAC_S0), U19.11 (S0)
- new net DAC_S1: U14.79 (DAC_S1), U19.10 (S1)
- new net DAC_S2: U14.80 (DAC_S2), U19.9 (S2)
- new net INA_ALERT_N: R76.2, U14.84 (INA_ALERT_N), U16.3 (Alert)
- new net INA_SCL: R80.2, U14.83 (INA_SCL), U16.5 (SCL)
- new net INA_SDA: R79.2, U14.82 (INA_SDA), U16.4 (SDA)
- new net MEAS_INHIBIT: R70.2, U14.5 (MEAS_INHIBIT), U17.6 (E_INHIBIT), U18.6 (E_INHIBIT)
- new net MEAS_S0: U14.2 (MEAS_S0), U17.11 (S0), U18.11 (S0)
- new net MEAS_S1: U14.3 (MEAS_S1), U17.10 (S1), U18.10 (S1)
- new net MEAS_S2: U14.4 (MEAS_S2), U17.9 (S2), U18.9 (S2)
- new net SHUNT_HIGH_SELECTED: U16.10 (VIN+), U17.3 (Z)
- new net SHUNT_LOW_SELECTED: U16.8 (VBUS), U16.9 (VIN-), U18.3 (Z)
- new net SPARE_IO_17: TP42.1, U14.17 (LAB_SCLK)
- new net SPARE_IO_33: TP43.1, U14.33 (LAB_MOSI)
- new net SPARE_IO_34: TP44.1, U14.34 (LAB_MISO)
- no-connect marks 12 -> 19
Other:
- removed sheet AG32 supervisor e strumenti
- note added: "0-3.3 V, common ground; calibrate before use."
- note added: "20 MHz | Controller clock"
- note added: "4051 | First measurement selector"
- note added: "4051 | Second measurement selector"
- note added: "A return path is required. Occupancy detection is assisted, not guaranteed."
- note added: "AG Base: U14 fitted, Lab components omitted, R56-R61 = 0R."
- note added: "AG UART0: TX pin68 / RX pin69. BOOT1 stays LOW via R84."
- note added: "AG32 section A | Experiment signals"
- note added: "AG32 section B | Port settings"
- note added: "AG32 section C | Board communication"
- note added: "AG32 section D | Current scan control"
- note added: "AG32 section F | Power and start-up"
- note added: "Adds Wi-Fi, Bluetooth and ESP32 project support."
- note added: "Adds Wi-Fi, Bluetooth and support for ESP32 projects."
- note added: "Applies a gentle test signal and watches how each connection responds."
- note added: "BOARD-TO-BOARD LINK"
- note added: "COMMUNICATION HUB"
- note added: "CONNECTIONS & POWER"
- note added: "CONTROL & LAB TOOLS"
- note added: "CURRENT MEASUREMENT"
- note added: "Chooses how each experiment port is connected."
- note added: "Chooses signal, power or ground for each port."
- note added: "Chooses which port is measured."
- note added: "Connect a circuit, choose how each port behaves, and explore what happens."
- note added: "Connect or disconnect the ESP32 from the experiment ports."
- note added: "Connects accessories directly to the optional ESP32."
- note added: "Connects compatible sensors with a small cable."
- note added: "Connects displays, cameras and other supported add-ons."
- note added: "Connects one side of the selected current sensor path."
- note added: "Connects or separates the ESP32 signals from the experiment."
- note added: "Connects the board to a computer."
- note added: "Connects the other side of the same sensor path."
- note added: "Connects this board to the shared CAN network."
- note added: "Creates the power used by the board."
- note added: "Current is measured separately by INA226."
- note added: "DIRECT ACCESS"
- note added: "ESP Base: U25 + R98-R102 fitted; U14, Lab and AG programming parts omitted."
- note added: "ESP32 PROGRAMS THE AG32"
- note added: "ESP32-S3 | Optional wireless module"
- note added: "Enables the end-of-network connection when needed."
- note added: "Exchanges data with the computer and other boards."
- note added: "Existing circuit preserved. Tester features require firmware and prototype validation; no new tester components were added."
- note added: "G3VM | Network end switch"
- note added: "GPIO47 TX / GPIO48 RX | GPIO15 BOOT0 | GPIO16 RESET (open-drain)"
- note added: "Give a port power or ground when selected."
- note added: "Gives each port a signal, power or ground connection."
- note added: "Gives the measurement circuits a stable voltage reference."
- note added: "INA226 | Current sensor"
- note added: "Internal DAC -> R77 -> selectable port. Read both sides of R77 with internal ADC."
- note added: "Keeps the controller running at a steady pace."
- note added: "Keeps the controller supply steady while it works."
- note added: "LIVE VIEW | SIX PORT VOLTAGES"
- note added: "LOCAL POWER SUPPORT"
- note added: "Lab: U14 + measurement components fitted. USB remains direct to ESP32."
- note added: "Lets this board exchange messages with the other boards."
- note added: "Links the controller to USB, the network and the optional ESP32."
- note added: "Loads the board controller without an external programmer."
- note added: "MAIN POWER"
- note added: "MEASURE | INTERNAL CONVERTERS"
- note added: "Measures the current of the selected port."
- note added: "NETWORK CONNECTION"
- note added: "Native ADC inputs remain on PORT_A0-A5."
- note added: "No external ADC, DAC, reference or op-amps."
- note added: "OPTION | ESP32-ONLY CONTROLLER"
- note added: "OPTIONAL ACCESSORY LINKS"
- note added: "OPTIONAL ESP32 MODULE"
- note added: "Observes all six ports while the experiment keeps running."
- note added: "Observes the ports and manages digital signals for the experiment."
- note added: "PORT LIGHTS"
- note added: "PORT MODE CONTROL"
- note added: "PORT SUPERVISOR"
- note added: "Passes power and communication to neighbouring boards."
- note added: "Powers, starts and provides access to the board controller."
- note added: "Provides the supply voltages used by supported accessories."
- note added: "Q3-Q8 | Electronic power switches"
- note added: "QWIIC ACCESSORIES"
- note added: "Reads the ports and handles digital signals."
- note added: "Recovery: keep ESP32 pins Hi-Z; use UART pads or the existing JTAG pads."
- note added: "SCAN | SMALL TEST SIGNALS"
- note added: "SIGNAL CONNECTIONS"
- note added: "SIX EXPERIMENT PORTS"
- note added: "SN65HVD230 | Network interface"
- note added: "SPAGHETTILAB | ONE BOARD, MANY POSSIBILITIES"
- note added: "SUPERVISOR START-UP"
- note added: "Scan: MOSFETs OFF, digital drivers Hi-Z, ESP switches OPEN, R77 bypass OFF."
- note added: "Selects one port at a time and measures the current flowing through it."
- note added: "Shows how the connected circuit changes over time."
- note added: "Shows the state of each port with coloured light."
- note added: "Six port voltages -> AG32 ADC"
- note added: "Starts the controller and provides programming access."
- note added: "TPS562201 | Main power supply"
- note added: "Turns the incoming power into the supply used by the board."
- note added: "U12 / U13 | Bidirectional signal switches"
- note added: "U14A-U14G are seven sections of ONE physical AG32 chip."
- note added: "USB CONNECTION"
- note added: "Uses AG32 to observe voltages without extra converter chips."
- note added: "Uses the ESP32 to configure the ports when AG32 is not fitted."
- note removed: "+1V5"
- note removed: "+2V8"
- note removed: "33k / 10k: nominal 3.302 V. Total load and thermal check required."
- note removed: "3V3 / R31"
- note removed: "A0 / GPIO7 — FILA 1"
- note removed: "A0-A5 = lato micro/J3; PORT_A0-A5 = lato MOSFET e J1/J140. Default aperto."
- note removed: "A1 / GPIO8 — FILA 2"
- note removed: "A2 / GPIO9 — FILA 3"
- note removed: "A3 / GPIO10 — FILA 4"
- note removed: "AG32 firmware: set all GPIO Hi-Z, disable both MOSFETs before switching modes. Analog bypass remains U12/U13."
- note removed: "AG32 universal board: ESP32 optional. See AG32 supervisor sheet and AG32-SUPERVISOR.md. Old TI/Q32 variants superseded on this branch."
- note removed: "AUXILIARY 1.5 V REGULATOR"
- note removed: "AUXILIARY 2.8 V REGULATOR"
- note removed: "BACKBONE"
- note removed: "BACKBONE MCU"
- note removed: "C79/C80: +2V8 decoupling. C81: +1V5 decoupling."
- note removed: "CAN AUTO TERMINAL RESISTOR CIRCUIT"
- note removed: "CAN TRANSCEIVER"
- note removed: "CLK_OUT"
- note removed: "CONNECTORS"
- note removed: "Check peripheral pinout, voltages and flex orientation."
- note removed: "DIRECT CLOCK - 3.3 V"
- note removed: "Defaults retained; optional GPIO links via R34/R35."
- note removed: "EXPANSION - 24-PIN FPC"
- note removed: "FPC BIAS RESISTORS"
- note removed: "FPC shares I2C on GPIO4/5; pull-ups to 3.3 V."
- note removed: "FPC signals, fixed bias pins and voltage limits: see project documentation."
- note removed: "FPC_PULLDOWN: 10k to GND"
- note removed: "FPC_PULLUP: 10k to +2V8"
- note removed: "Fit only for a verified peripheral. R31-R35: DNP in camera profile."
- note removed: "Fixed auxiliary rails: 2.8 V / 1.5 V. Check peripheral voltage requirements."
- note removed: "GND"
- note removed: "GPIO mode: /OE=0, P=OFF, N=OFF. 3V3/GND mode: /OE=1 prima di abilitare il MOSFET."
- note removed: "GPIO1"
- note removed: "GPIO17"
- note removed: "GPIO18"
- note removed: "GPIO2"
- note removed: "GPIO21"
- note removed: "GPIO38"
- note removed: "GPIO39"
- note removed: "GPIO3: RESET, open-drain only; JTAG strap."
- note removed: "GPIO40"
- note removed: "GPIO41"
- note removed: "GPIO42"
- note removed: "GPIO46: standby; boot strap, keep low at reset."
- note removed: "GPIO6"
- note removed: "IMPLEMENTATO: solo GPIO/3V3/GND. INA, shunt, DAC e lettura ADC dedicata rimandati."
- note removed: "ISOLAMENTO BIDIREZIONALE J3 <-> J1/J140 — /OE=1 APERTO, /OE=0 COLLEGATO"
- note removed: "Input: VCORE 3.3 V. Place capacitors close to the LDO."
- note removed: "J1/J140: PORT_A0-A5. J3: lato micro diretto. GPIO13/14: comandi isolamento."
- note removed: "J3: 3V3/GND + A0/A1; 3V3/GND + A2/A3; 3V3/GND + A4/A5"
- note removed: "Keep VIN bypass, bootstrap and SW loop short."
- note removed: "MODULE BAY 0"
- note removed: "NON attivare P e N insieme. Questa revisione non aggiunge limitazione hardware."
- note removed: "OPTIONAL FPC CONNECTIONS - 0R LINKS, DNP BY DEFAULT"
- note removed: "PIN CONFIG RGB LEDs"
- note removed: "PORTE UNIVERSALI A0-A5 — BASE GPIO / 3V3 / GND"
- note removed: "PORT_A4 / GPIO1 — FILA 5"
- note removed: "PORT_A5 / GPIO2 — FILA 6"
- note removed: "PULLDOWN"
- note removed: "PULLUP"
- note removed: "Q3-Q8: A=P-channel; B=N-channel. U11 A-F: comandi, G: alimentazione/I2C."
- note removed: "QWIIC EXPANSION - 3.3 V"
- note removed: "R35: only if peripheral accepts 3.3 V control."
- note removed: "RX44 / R33"
- note removed: "SCL"
- note removed: "SDA"
- note removed: "Shared 3.3 V: ESP32-S3, LEDs, peripherals and camera LDO inputs."
- note removed: "TX43 / R32"
- note removed: "U11: indirizzo I2C 0x20. Tutti i gate spenti al reset tramite pull-up P / pull-down N."
- note removed: "UART0 shared with debug; TX may emit boot logs."
- note removed: "USB"
- note removed: "VCORE also supplies LEDs: check total load and temperature."
- note removed: "VCORE: 5 V TO 3.3 V / 2 A BUCK"
- title: (none) -> SpaghettiLab — functional overview
- moved on the sheet: C1, C11, C5, C74, C84, C85, C86, C88, C89, C9, D6, H1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

Commit message: Finalize AG32 backbone layout, sensor pinout and routing setup
Parts:
- added J5: FH12-24S-0.5SH(55), SpaghettiLAB:Hirose_FH12-24S-0.5SH_1x24-1MP_P0.50mm_Horizontal, symbol SpaghettiLAB:FPC_24_Hirose_FH12
Connections:
- net A0: now also J3.7; no longer J3.3
- net A1: now also J3.1; no longer J3.4
- net A2: now also J3.12; no longer J3.7
- net A3: now also J3.10; no longer J3.8
- net A4: now also J3.8; no longer J3.11
- net A5: now also J3.6; no longer J3.12
- net DAC1_SPARE: now also J5.22
- net GND: now also J3.4, J3.5, J3.9, J5.1, J5.10, J5.14, J5.24, J5.6; no longer J3.10, J3.2, J3.6
- net IO11: now also J5.4
- net IO12: now also J5.5
- net IO17: now also J5.7
- net IO18: now also J5.8
- net IO21: now also J5.9
- net IO38: now also J5.11
- net IO39: now also J5.12
- net IO4: now also J5.17
- net IO40: now also J5.13
- net IO41: now also J5.15
- net IO42: now also J5.16
- net IO5: now also J5.18
- net IO6: now also J5.3
- net SPARE_IO_17: now also J5.19
- net SPARE_IO_33: now also J5.20
- net SPARE_IO_34: now also J5.21
- net VCORE: now also J3.11, J3.2, J3.3, J5.2, J5.23; no longer J3.1, J3.5, J3.9
- net AG_USB_DM renamed USB_AG_D-
- net AG_USB_DP renamed USB_AG_D+
- net Net-(U19-USB_D+) renamed USB_ESP_D+
- net Net-(U19-USB_D-) renamed USB_ESP_D-
Other:
- note added: "Connects extra modules through a flat cable at the board edge."
- note added: "ESP GPIO + Qwiic + 4 AG32 signals. 3.3 V only."
- note added: "EXPAND | ESP32 GPIO"
- note added: "GPIO35-37 reserved for PSRAM."
- note added: "GPIO39-42 share JTAG."
- note added: "J5: ESP32 + AG32 expansion"
- note removed: "0-3.3 V, common ground; calibrate before use."
- note removed: "Gives the measurement circuits a stable voltage reference."
- note removed: "MEASURE | INTERNAL CONVERTERS"
- note removed: "Provides the supply voltages used by supported accessories."
- note removed: "Six port voltages -> AG32 ADC"
- note removed: "Uses AG32 to observe voltages without extra converter chips."
